File: Voyager40.sch (KiCad schematic (older format))
At the start: 190 parts, among them Q1 2N7002, SW1 5.2x5.2mm, U1 ATmega32U2-AU, U2 PRTR5V0U2X, Y1 16Mhz

Commit message: Initial STM32F072CB replacement
Parts:
- removed C2: 10uF, Capacitors_SMD:C_0603, symbol Device:C_Small
- removed C3, C4: 0.1uF, Capacitors_SMD:C_0603, symbol Device:C_Small
- removed C6: 1uF, Capacitors_SMD:C_0603, symbol Device:C_Small
- removed C7, C8: 22pF, Capacitors_SMD:C_0603, symbol Device:C_Small
- removed R67, R68: 22, Resistors_SMD:R_0805, symbol Device:R_Small
- removed R70: 10k, Resistors_SMD:R_0805, symbol Device:R_Small
- removed R71: 1k, Resistors_SMD:R_0805, symbol Device:R_Small
- removed SW1: 5.2x5.2mm, random-keyboard-parts:SKQGADE010, symbol Voyager60-rescue:SW_Push
- removed U1: ATmega32U2-AU, Housings_DFN_QFN:QFN-32-1EP_5x5mm_Pitch0.5mm, symbol MCU_Microchip_ATmega:ATmega32U2-AU
- removed Y1: 16Mhz, Crystals:Crystal_SMD_3225-4pin_3.2x2.5mm, symbol Device:Crystal_GND24
- added C19, C20, C21, C22: 0.1uF, Capacitors_SMD:C_0603, symbol Device:C_Small
- added C23, C24: 4.7uF, Capacitors_SMD:C_0603, symbol Device:C_Small
- added C25, C26: 1uF, Capacitors_SMD:C_0603, symbol Device:C_Small
- added R2: 10k, Resistors_SMD:R_0805, symbol Device:R_Small
- added R3: 5.1k, Resistors_SMD:R_0805, symbol Device:R_Small
- added SW2: SW_Push, Buttons_Switches_SMD:SW_SPST_SKQG, symbol Switch:SW_Push
- added SW3: SW_SPDT, Buttons_Switches_SMD:SW_SPDT_PCM12, symbol Switch:SW_SPDT
- added U3: STM32F072CBUx, Housings_DFN_QFN:QFN-48-1EP_7x7mm_Pitch0.5mm, symbol MCU_ST_STM32F0:STM32F072CBUx
- added U4: MCP1700-3002E_SOT23, TO_SOT_Packages_SMD:SOT-23, symbol Regulator_Linear:MCP1700-3002E_SOT23
- R69: value 1k -> 100
Connections:
- net labels added: +3V3, SWCLK, SWDIO
- wire segments 533 -> 534
- no-connect marks 1 -> 8
Other:
- moved on the sheet: Q1, R69
