File: Voyager40.sch (KiCad schematic (older format))
At the start: 190 parts, among them Q1 2N7002, SW1 5.2x5.2mm, U1 ATmega32U2-AU, U2 PRTR5V0U2X, Y1 16Mhz

Commit message: Repair the column traces
Parts:
- SW1: symbol Voyager60-rescue:SW_Push -> Voyager40-rescue:SW_Push-Voyager60-rescue
- U1: symbol MCU_Microchip_ATmega:ATmega32U2-AU -> Voyager40-rescue:ATmega32U2-AU-MCU_Microchip_ATmega
Changed lines of the file:
@@
 $EndComp
 $Comp
-L Voyager60-rescue:SW_Push SW1
+L Voyager40-rescue:SW_Push-Voyager60-rescue SW1
 U 1 1 5B323AA5
 P 6125 7300
@@
 $EndComp
 $Comp
-L MCU_Microchip_ATmega:ATmega32U2-AU U1
+L Voyager40-rescue:ATmega32U2-AU-MCU_Microchip_ATmega U1
 U 1 1 5D0B79E1
 P 7475 8400
@@
 Text GLabel 8175 8700 2    50   Input ~ 0
 ROW3
+Text GLabel 8175 8400 2    50   Input ~ 0
+COL1
+Text GLabel 8175 8300 2    50   Input ~ 0
+COL0
 $EndSCHEMATC
